File: myportion-kicad/myportion-kicad.kicad_pcb (KiCad board)
At the start: 2 copper layers, 2 parts

Commit message: Add rough kicad project
Parts:
- added P1: RFID-RC522-MODULE, RF_Module:nRF24L01_Breakout, F.Cu at (147.3, 86.4)
- added R1: R_Variable, Package_TO_SOT_THT:TO-3PB-3_Horizontal_TabDown, F.Cu at (166.4, 86.4)
- added R2: R, Resistor_SMD:R_4020_10251Metric_Pad1.65x5.30mm_HandSolder, F.Cu at (156.2, 83.8)
- added U1: NodeMCU_1.0_(ESP-12E), Connector_Hirose:Hirose_DF12_DF12E3.0-32DP-0.5V_2x16_P0.50mm_Vertical, F.Cu at (146.6, 65.1)
- moved A1 45.6 mm to (165.1, 36.8)
- moved A2 2.90 mm to (139.7, 49.5), turned to 90 degrees
Routing:
- net GND: track 0.00 -> 45.2 mm, vias 0 -> 2
- net Net-(A1-Pad15): track 0.00 -> 44.6 mm
- net Net-(A1-Pad16): track 0.00 -> 44.0 mm
- net Net-(A2-Pad13): track 0.00 -> 43.6 mm
- net Net-(A2-Pad16): track 0.00 -> 28.0 mm
- net Net-(R1-Pad2): track 0.00 -> 27.7 mm, vias 0 -> 2
- net Net-(A2-Pad14): track 0.00 -> 27.6 mm
- net Net-(A2-Pad15): track 0.00 -> 27.1 mm
- net Net-(P1-Pad2): track 0.00 -> 24.6 mm
- net Net-(P1-Pad6): track 0.00 -> 24.5 mm
- net Net-(P1-Pad4): track 0.00 -> 17.9 mm
- net Net-(P1-Pad5): track 0.00 -> 15.7 mm, vias 0 -> 2
- net Net-(P1-Pad8): track 0.00 -> 12.3 mm
- net Net-(A1-Pad14): track 0.00 -> 0.70 mm
